File: hardware/FCU/FCU.kicad_pcb (KiCad board)
At the start: 2 copper layers, 80 x 62.2 mm, 37 parts, among them J1 Valve Power 12V, J2 Valve Ctrl, J3 Sensor, J4 OLED Display, P1 Power In, P2 + in, P3 3.3V out, P4 - in, P5 - out, P6 Buttons, Q1 IRLZ44N, Q2 IRLZ44N, Q3 IRLZ44N, Q4 IRLZ44N

Commit message: Add hardware READMEs for FCU and RCU
Parts:
- R10: footprint Diode_THT:D_A-405_P2.54mm_Vertical_AnodeUp -> Resistor_THT:R_Axial_DIN0207_L6.3mm_D2.5mm_P2.54mm_Vertical
Changed lines of the file:
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@@
 		(sheetname "/")
 		(sheetfile "FCU.kicad_sch")
+		(units
+			(unit
+				(name "A")
+				(pins "1" "2")
+			)
+		)
 		(attr through_hole)
 		(duplicate_pad_numbers_are_jumpers no)
@@
 		)
 	)
-	(footprint "Diode_THT:D_A-405_P2.54mm_Vertical_AnodeUp"
+	(footprint "Resistor_THT:R_Axial_DIN0207_L6.3mm_D2.5mm_P2.54mm_Vertical"
 		(layer "F.Cu")
 		(at 144.78 87.63 -90)
-		(descr "Diode, A-405 series, Axial, Vertical, pin pitch=2.54mm, length*diameter=5.2*2.7mm^2, http://www.diodes.com/_files/packages/A-405.pdf")
-		(tags "Diode A-405 series Axial Vertical pin pitch 2.54mm  length 5.2mm diameter 2.7mm")
+		(descr "Resistor, Axial_DIN0207 series, Axial, Vertical, pin pitch=2.54mm, 0.25W = 1/4W, length*diameter=6.3*2.5mm^2, http://cdn-reichelt.de/documents/datenblatt/B400/1_4W%23YAG.pdf")
+		(tags "Resistor Axial_DIN0207 series Axial Vertical pin pitch 2.54mm 0.25W = 1/4W length 6.3mm diameter 2.5mm")
 		(property "Reference" "R10"
-			(at 1.27 -2.47 270)
+			(at 1.27 -2.37 90)
 			(layer "F.SilkS")
 			(effects
@@
 		)
 		(property "Value" "10k"
-			(at 1.27 3.359 270)
+			(at 1.27 2.37 90)
 			(layer "F.Fab")
 			(effects
@@
 		)
 		(property "Datasheet" ""
-			(at 0 0 270)
+			(at 0 0 90)
 			(layer "F.Fab")
 			(hide yes)
@@
 		)
 		(property "Description" ""
-			(at 0 0 270)
+			(at 0 0 90)
 			(layer "F.Fab")
 			(hide yes)
@@
 			)
 		)
-		(property "KiLib_Generator" "diode/THT"
-			(at 0 0 270)
+		(property "KiLib_Generator" "resistor/THT"
+			(at 0 0 90)
 			(layer "F.SilkS")
 			(hide yes)
@@
 		(sheetname "/")
 		(sheetfile "FCU.kicad_sch")
+		(units
+			(unit
+				(name "A")
+				(pins "1" "2")
+			)
+		)
 		(attr through_hole)
 		(duplicate_pad_numbers_are_jumpers no)
-		(fp_arc
-			(start 1.058537 1.02)
-			(mid -1.47 0)
-			(end 1.058537 -1.02)
+		(fp_line
+			(start 1.37 0)
+			(end 1.44 0)
 			(stroke
 				(width 0.12)
@@
 			(layer "F.SilkS")
 		)
+		(fp_circle
+			(center 0 0)
+			(end 1.37 0)
+			(stroke
+				(width 0.12)
+				(type solid)
+			)
+			(fill no)
+			(layer "F.SilkS")
+		)
 		(fp_rect
-			(start -1.6 -1.6)
-			(end 3.69 1.6)
+			(start -1.5 -1.5)
+			(end 3.59 1.5)
 			(stroke
 				(width 0.05)
@@
 		(fp_circle
 			(center 0 0)
-			(end 1.35 0)
+			(end 1.25 0)
 			(stroke
 				(width 0.1)
@@
 			(layer "F.Fab")
 		)
-		(fp_text user "A"
-			(at 4.44 0 270)
-			(layer "F.SilkS")
-			(effects
-				(font
-					(size 1 1)
-					(thickness 0.15)
-				)
-			)
-		)
-		(fp_text user "A"
-			(at 4.44 0 270)
-			(layer "F.Fab")
-			(effects
-				(font
-					(size 1 1)
-					(thickness 0.15)
-				)
-			)
-		)
 		(fp_text user "${REFERENCE}"
-			(at 1.27 -2.47 270)
+			(at 1.27 -2.37 90)
 			(layer "F.Fab")
 			(effects
@@
 			)
 		)
-		(pad "1" thru_hole roundrect
+		(pad "1" thru_hole circle
 			(at 0 0 270)
-			(size 1.8 1.8)
-			(drill 0.9)
+			(size 1.6 1.6)
+			(drill 0.8)
 			(layers "*.Cu" "*.Mask")
 			(remove_unused_layers no)
-			(roundrect_rratio 0.138889)
 			(net "/Button_Up")
 			(pintype "passive")
@@
 		(pad "2" thru_hole circle
 			(at 2.54 0 270)
-			(size 1.8 1.8)
-			(drill 0.9)
+			(size 1.6 1.6)
+			(drill 0.8)
 			(layers "*.Cu" "*.Mask")
 			(remove_unused_layers no)
@@
 		)
 		(embedded_fonts no)
-		(model "${KICAD10_3DMODEL_DIR}/Diode_THT.3dshapes/D_A-405_P2.54mm_Vertical_AnodeUp.step"
+		(model "${KICAD10_3DMODEL_DIR}/Resistor_THT.3dshapes/R_Axial_DIN0207_L6.3mm_D2.5mm_P2.54mm_Vertical.step"
 			(offset
 				(xyz 0 0 0)
@@
 	)
 	(segment
+		(start 140.97 74.93)
+		(end 142.24 73.66)
+		(width 2)
+		(layer "B.Cu")
+		(net "Net-(D5-A)")
+	)
+	(segment
+		(start 142.24 73.66)
+		(end 142.24 67.31)
+		(width 2)
+		(layer "B.Cu")
+		(net "Net-(D5-A)")
+	)
+	(segment
 		(start 86.36 85.09)
 		(end 90.17 85.09)
@@
 		(net "unconnected-(J2-Pin_4-Pad4)")
 	)
-	(segment
-		(start 140.97 74.93)
-		(end 142.24 73.66)
-		(width 2)
-		(layer "B.Cu")
-		(net "Net-(D5-A)")
-	)
-	(segment
-		(start 142.24 73.66)
-		(end 142.24 67.31)
-		(width 2)
-		(layer "B.Cu")
-		(net "Net-(D5-A)")
-	)
 	(embedded_fonts no)
