File: hardware/FCU/FCU.kicad_sch (KiCad schematic)
At the start: 37 parts, among them J1 Valve Power 12V, J2 Valve Ctrl, J3 Sensor, J4 OLED Display, P1 Power In, P2 + in, P3 3.3V out, P4 - in, P5 - out, P6 Buttons, Q1 IRLZ44N, Q2 IRLZ44N, Q3 IRLZ44N, Q4 IRLZ44N

Commit message: Add hardware READMEs for FCU and RCU
Parts:
- R10: footprint Diode_THT:D_A-405_P2.54mm_Vertical_AnodeUp -> Resistor_THT:R_Axial_DIN0207_L6.3mm_D2.5mm_P2.54mm_Vertical; KiLib_Generator diode/THT -> resistor/THT
Other:
- title: AirSuspension Controller -> AirSuspension Fron Control Unit
Changed lines of the file:
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@@
 	(paper "A4")
 	(title_block
-		(title "AirSuspension Controller")
+		(title "AirSuspension Fron Control Unit")
 		(rev "0.01")
+		(comment 1 "MCU, Power and Valve drivers")
 	)
 	(rectangle
@@
 			)
 		)
-		(property "Footprint" "Diode_THT:D_A-405_P2.54mm_Vertical_AnodeUp"
+		(property "Footprint" "Resistor_THT:R_Axial_DIN0207_L6.3mm_D2.5mm_P2.54mm_Vertical"
 			(at 237.998 69.85 90)
 			(hide yes)
@@
 			)
 		)
-		(property "KiLib_Generator" "diode/THT"
+		(property "KiLib_Generator" "resistor/THT"
 			(at 236.22 69.85 0)
 			(hide yes)
