File: hardware/RCU/RCU.kicad_sch (KiCad schematic)
At the start: 19 parts, among them J1 Sensor, J2 DE9_Pins, J3 Valves, J4 InputConnector IP68, J5 Spare, P2 + in, P3 5V out, P4 - in, P5 - out

Commit message: Add hardware READMEs for FCU and RCU
Other:
- title: (none) -> Rear Control Unit
Changed lines of the file:
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@@
 	(generator_version "10.0")
 	(paper "A4")
+	(title_block
+		(title "Rear Control Unit")
+		(comment 1 "Connector Distribution")
+		(comment 2 "Sensor power, Level shifter")
+	)
 	(rectangle
 		(start 193.9132 28.8925)
